File: hardware/AppsecPnw-2024.kicad_pcb (KiCad board)
At the start: 2 copper layers, 75.2 x 76.5 mm, 49 parts, among them J1 OLED, J2 Battery, J3 Conn_02x03_Odd_Even, J5 UART, P1 USB_C_Plug_USB2.0, Q1 DMG3415U-7, SW1 ON, SW2 LEFT, SW3 DOWN, SW4 UP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

Commit message: feat(hw): add tickness
Other:
- board text added: "PCB tickness = 0.8 mm"
- board text added: "PCB tickness = 1.0 mm"

Commit message: fix(Hw): fix dimensions layers and delete duplicated PCB thickness note
Other:
- board text removed: "PCB tickness = 0.8 mm"

Commit message: fix(Hw): Change PCB and pull up resistor for boot added
Parts:
- added R5: 3.3K, Resistor_SMD:R_0603_1608Metric, B.Cu at (188.4, 44.5)
- F1: value 0.5A -> 1A
Connections:
- U2 pad 10: unconnected-(U2-IO8-Pad10) -> /IO8
Routing:
- net +3V3: track 184.9 -> 200.5 mm
- net /IO8: track 0.00 -> 3.82 mm
- net GND: track 52.3 -> 54.2 mm

Commit message: feat(): add labels
Parts:
- removed kibuzzard-660EEC06: G***, kibuzzard-660EEC06
- removed kibuzzard-660EEC1C: G***, kibuzzard-660EEC1C
- removed kibuzzard-660EEC32: G***, kibuzzard-660EEC32
- removed kibuzzard-660EEC49: G***, kibuzzard-660EEC49
- added kibuzzard-663AC028: G***, kibuzzard-663AC028, B.Cu at (232.0, 50.5)
- added kibuzzard-663AC038: G***, kibuzzard-663AC038, B.Cu at (233.4, 53.1)
- added kibuzzard-663AC049: G***, kibuzzard-663AC049, B.Cu at (233.4, 55.6)
- added kibuzzard-663AC054: G***, kibuzzard-663AC054, B.Cu at (233.2, 58.1)
- moved kibuzzard-6616FF4C 0.31 mm to (229.9, 58.7)
Other:
- board text added: "github.com/ElectronicCats/ Badge-AppsecPnw-2024"
- board text added: "v2.1"
- board text added: "youtu.be/dQw4w9WgXcQ?si=zUtmE9e61LVhIf0K"
- board text removed: "v2.0"
